Commit message: add gazebo model

File: robotiq_s_model_visualization/cfg/s-model_articulated.xacro (robot description, xacro)
@@ -6,5 +6,8 @@
 <robot name="s-model_articulated" xmlns:xacro="http://ros.org/wiki/xacro">
 	<xacro:include filename="$(find robotiq_s_model_visualization)/cfg/s-model_articulated_macro.xacro" />
-	<xacro:s-model_articulated prefix=""/>
+	<xacro:s-model_articulated prefix=""
+	                           fixed_joints="revolute"
+	                           default_joint2="-0.52"
+	                           default_joint3="0.0" />
 <!--
 	<include filename="$(find robotiq_s_model_visualization)/cfg/s-model_finger_articulated_macro.xacro" />

File: robotiq_s_model_visualization/cfg/s-model_articulated_macro.xacro (robot description, xacro)
@@ -7,8 +7,11 @@
 <robot xmlns:xacro="http://ros.org/wiki/xacro">
 	<xacro:include filename="$(find robotiq_s_model_visualization)/cfg/s-model_finger_articulated_macro.xacro" />
-	<xacro:macro name="s-model_articulated" params="prefix">
-	<xacro:s-model_finger_articulated prefix="${prefix}finger_1_"/>
-	<xacro:s-model_finger_articulated prefix="${prefix}finger_2_"/>
-	<xacro:s-model_finger_articulated prefix="${prefix}finger_middle_"/>
+	<xacro:macro name="s-model_articulated" params="prefix fixed_joints default_joint2 default_joint3">
+	<xacro:s-model_finger_articulated prefix="${prefix}finger_1_"
+	                                  fixed_joints="${fixed_joints}" default_joint2="${default_joint2}" default_joint3="${default_joint3}" />
+	<xacro:s-model_finger_articulated prefix="${prefix}finger_2_"
+	                                  fixed_joints="${fixed_joints}" default_joint2="${default_joint2}" default_joint3="${default_joint3}" />
+	<xacro:s-model_finger_articulated prefix="${prefix}finger_middle_"
+	                                  fixed_joints="${fixed_joints}" default_joint2="${default_joint2}" default_joint3="${default_joint3}" />
 		<!-- link list -->
 		<link name="${prefix}palm">

File: robotiq_s_model_visualization/cfg/s-model_finger_articulated_macro.xacro (robot description, xacro)
@@ -6,5 +6,5 @@
 -->
 <robot xmlns:xacro="http://ros.org/wiki/xacro">
-	<xacro:macro name="s-model_finger_articulated" params="prefix">
+	<xacro:macro name="s-model_finger_articulated" params="prefix fixed_joints default_joint2 default_joint3">
 		<!-- link list -->
 		<link name="${prefix}link_0">
@@ -109,20 +109,20 @@
 			<axis xyz="0 0 1"/>
 			<origin xyz="0.020 0 0" rpy="0 0 0"/>
+			<limit lower="0" upper="2.0944" effort="100" velocity="100"/>
+		</joint>
+		<!-- WARNING: LIMITS NOT CORRECT -->
+		<joint name="${prefix}joint_2" type="${fixed_joints}">
+			<parent link="${prefix}link_1"/>
+			<child link="${prefix}link_2"/>
+			<axis xyz="0 0 1"/>
+			<origin xyz="0.050 -.028 0" rpy="0 0 ${default_joint2}"/>
 			<limit lower="0" upper="3.1416" effort="100" velocity="100"/>
 		</joint>
 		<!-- WARNING: LIMITS NOT CORRECT -->
-		<joint name="${prefix}joint_2" type="revolute">
-			<parent link="${prefix}link_1"/>
-			<child link="${prefix}link_2"/>
-			<axis xyz="0 0 1"/>
-			<origin xyz="0.050 -.028 0" rpy="0 0 -0.52"/>
-			<limit lower="0" upper="3.1416" effort="100" velocity="100"/>
-		</joint>
-		<!-- WARNING: LIMITS NOT CORRECT -->
-		<joint name="${prefix}joint_3" type="revolute">
+		<joint name="${prefix}joint_3" type="${fixed_joints}">
 			<parent link="${prefix}link_2"/>
 			<child link="${prefix}link_3"/>
 			<axis xyz="0 0 1"/>
-			<origin xyz="0.039 0 0" rpy="0 0 0"/>
+			<origin xyz="0.039 0 0" rpy="0 0 ${default_joint3}"/>
 			<limit lower="0" upper="3.1416" effort="100" velocity="100"/>
 		</joint>
